File: pcb/control-module.kicad_pcb (KiCad board)
At the start: 2 copper layers, 50.3 x 37.8 mm, 63 parts, among them J1 Screw_Terminal_01x08, J2 Conn_01x06_Pin, J3 USB_C_Receptacle_USB2.0_16P, J4 Micro_SD_Card, J5 Screw_Terminal_01x02, Q1 SiS454DN, Q2 SiS454DN, Q3 SiS454DN, SW1 SW_DIP_x03, U1 TC2185-3.3VxCTTR, U2 USBLC6-2SC6, U3 STM32U545RETxQ, U4 MS5607-02BA, U5 LSM6DSL

Commit message: Changed pin order on recovery connections
Connections:
- J1 pad 1: /Recovery Power -> /Valve Controller/Out
- J1 pad 2: /Valve Controller/Out -> /Recovery Power
- J1 pad 3: /Recovery Power -> /Pyro Controller 1/Out
- J1 pad 4: /Pyro Controller 1/Out -> /Recovery Power
- J1 pad 5: /Recovery Power -> /Pyro Controller 2/Out
- J1 pad 6: /Pyro Controller 2/Out -> /Recovery Power
Changed lines of the file:
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@@
 			(remove_unused_layers no)
 			(roundrect_rratio 0.113636)
-			(net 88 "/Recovery Power")
+			(net 40 "/Valve Controller/Out")
 			(pinfunction "Pin_1")
 			(pintype "passive")
@@
 			(layers "*.Cu" "*.Mask")
 			(remove_unused_layers no)
-			(net 40 "/Valve Controller/Out")
+			(net 88 "/Recovery Power")
 			(pinfunction "Pin_2")
 			(pintype "passive")
@@
 			(layers "*.Cu" "*.Mask")
 			(remove_unused_layers no)
-			(net 88 "/Recovery Power")
+			(net 39 "/Pyro Controller 1/Out")
 			(pinfunction "Pin_3")
 			(pintype "passive")
@@
 			(layers "*.Cu" "*.Mask")
 			(remove_unused_layers no)
-			(net 39 "/Pyro Controller 1/Out")
+			(net 88 "/Recovery Power")
 			(pinfunction "Pin_4")
 			(pintype "passive")
@@
 			(layers "*.Cu" "*.Mask")
 			(remove_unused_layers no)
-			(net 88 "/Recovery Power")
+			(net 38 "/Pyro Controller 2/Out")
 			(pinfunction "Pin_5")
 			(pintype "passive")
@@
 			(layers "*.Cu" "*.Mask")
 			(remove_unused_layers no)
-			(net 38 "/Pyro Controller 2/Out")
+			(net 88 "/Recovery Power")
 			(pinfunction "Pin_6")
 			(pintype "passive")
