File: pcb/control-module.kicad_pcb (KiCad board)
At the start: 2 copper layers, 50.3 x 37.8 mm, 63 parts, among them J1 Screw_Terminal_01x08, J2 Conn_01x06_Pin, J3 USB_C_Receptacle_USB2.0_16P, J4 Micro_SD_Card, J5 Screw_Terminal_01x02, Q1 SiS454DN, Q2 SiS454DN, Q3 SiS454DN, SW1 SW_DIP_x03, U1 TC2185-3.3VxCTTR, U2 USBLC6-2SC6, U3 STM32U545RETxQ, U4 MS5607-02BA, U5 LSM6DSL

Commit message: Revision 1
Parts:
- removed R4, R5, R6: 10k, Resistor_SMD:R_0603_1608Metric_Pad0.98x0.95mm_HandSolder
- added D4: B350A-13-F, Diode_SMD:D_SOD-123F, F.Cu at (122.0, 61.8)
- added JP2: SolderJumper_2_Open, Jumper:SolderJumper-2_P1.3mm_Open_RoundedPad1.0x1.5mm, F.Cu at (130.0, 80.5)
- added RN1: 10k, Resistor_SMD:R_Array_Convex_4x0612, F.Cu at (149.6, 83.3)
- added RN2: 10k, Resistor_SMD:R_Array_Convex_4x0612, F.Cu at (153.7, 58.4)
- J2: footprint Connector_PinHeader_2.54mm:PinHeader_1x06_P2.54mm_Vertical -> Connector_PinHeader_2.54mm:PinHeader_1x07_P2.54mm_Vertical
- moved R13 5.78 mm to (126.2, 57.9)
- moved R15 5.20 mm to (128.8, 63.8)
- moved G*** 4.51 mm to (140.7, 76.2)
- moved R14 3.88 mm to (126.2, 59.4), turned to 180 degrees
- moved R16 3.68 mm to (128.8, 59.6), turned to -90 degrees
- moved D2 3.30 mm to (150.9, 80.3)
- moved R3 3.30 mm to (149.1, 80.3)
- moved Q2 1.88 mm to (126.2, 62.5), turned to -90 degrees
- moved JP1 1.52 mm to (151.5, 87.6)
- moved C18 1.42 mm to (129.0, 71.1), turned to 90 degrees
- moved J2 1.27 mm to (132.8, 87.6)
- moved R1 1.05 mm to (126.0, 80.5), turned to 0 degrees
- moved C6 0.92 mm to (133.1, 66.3), turned to 180 degrees
- moved C19 0.30 mm to (129.5, 77.7)
- moved C17 0.25 mm to (132.6, 80.9)
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Connections:
- net /MCU/VDDA renamed VDDA
- J2 pad 5: GNDA -> +BATT
- R10 pad 1: /Pyro Controller 2/Fire -> /MCU/PYRO2_FIRE
- R11 pad 1: /Pyro Controller 2/Continutity -> /MCU/ADC1_IN6
- R12 pad 2: /Pyro Controller 2/Continutity -> /MCU/ADC1_IN6
- R13 pad 2: /Valve Controller/Fire -> /MCU/VALVE_FIRE
- R14 pad 1: /Valve Controller/Fire -> /MCU/VALVE_FIRE
- R15 pad 1: /Valve Controller/Continutity -> /MCU/ADC1_IN15
- R16 pad 2: /Valve Controller/Continutity -> /MCU/ADC1_IN15
- R17 pad 2: /Pyro Controller 1/Fire -> /MCU/PYRO1_FIRE
- R18 pad 1: /Pyro Controller 1/Fire -> /MCU/PYRO1_FIRE
- R19 pad 1: /Pyro Controller 1/Continutity -> /MCU/ADC1_IN5
- R20 pad 2: /Pyro Controller 1/Continutity -> /MCU/ADC1_IN5
- R9 pad 2: /Pyro Controller 2/Fire -> /MCU/PYRO2_FIRE
- SW1 pad 5: unconnected-(SW1-Pad5) -> Net-(RN2-R4.2)
- U3 pad 14: unconnected-(U3-PA0-Pad14) -> /MCU/ADC1_IN5
- U3 pad 15: /IMU Sensors/pres_sclk -> /MCU/ADC1_IN6
- U3 pad 16: unconnected-(U3-PA2-Pad16) -> /MCU/PYRO2_FIRE
- U3 pad 2: unconnected-(U3-PC13-Pad2) -> /MCU/VALVE_FIRE
- U3 pad 21: unconnected-(U3-PA5-Pad21) -> /IMU Sensors/pres_sclk
- U3 pad 24: unconnected-(U3-PB0-Pad24) -> /MCU/ADC1_IN15
- U3 pad 25: unconnected-(U3-PB1-Pad25) -> /Bat Sense
- U3 pad 5: unconnected-(U3-PH0-Pad5) -> /MCU/PYRO1_FIRE
Routing:
- net /MCU/ADC1_IN15: track 0.00 -> 29.6 mm, vias 0 -> 2
- net /MCU/ADC1_IN5: track 0.00 -> 20.1 mm, vias 0 -> 2
- net /MCU/VALVE_FIRE: track 0.00 -> 19.6 mm, vias 0 -> 2
- net /MCU/ADC1_IN6: track 0.00 -> 16.6 mm, vias 0 -> 2
- net /Valve Controller/Out: track 0.00 -> 12.9 mm
- net /MCU/PYRO2_FIRE: track 0.00 -> 12.5 mm, vias 0 -> 2
- net /MCU/PYRO1_FIRE: track 0.00 -> 12.1 mm, vias 0 -> 2
- net /Bat Sense: track 0.00 -> 11.7 mm, vias 0 -> 2
- net GNDA: track 14.4 -> 23.9 mm
- net /Pyro Controller 1/Out: track 0.00 -> 9.36 mm
- net +BATT: track 0.00 -> 8.65 mm
- net /Pyro Controller 2/Out: track 0.00 -> 8.48 mm
- net GNDD: track 28.7 -> 34.3 mm, vias 35 -> 53
- net VDDA: track 0.00 -> 5.59 mm
- net /IMU Sensors/imu_int2: track 7.87 -> 13.0 mm, vias 0 -> 2
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Other:
- board text added: "+12V"
- board text added: "+3.3V"
- board text added: "BAT+"
- board text added: "Control Module Rev. 1"
- board text added: "Energize"
- board text added: "GNDA"
- board text added: "P1+"
- board text added: "P1-"
- board text added: "P2+"
- board text added: "P2-"
- board text added: "V+"
- board text added: "V-"
- board text added: "X Eject Boot Reset"
- board text removed: "Ride-Along Module Rev. 1"
