File: pcb/STM32U545RETxQ.kicad_sch (KiCad schematic)
At the start: 14 parts, among them U3 STM32U545RETxQ

Commit message: Revision 1
Connections:
- net SPI1_SCK: now also U3.21 (PA5); no longer U3.15 (PA1)
- net ADC1_IN5: now reaches U3.14 (PA0)
- net PYRO2_FIRE: now reaches U3.16 (PA2)
- net VALVE_FIRE: now reaches U3.2 (PC13)
- net ADC1_IN15: now reaches U3.24 (PB0)
- net ADC1_IN16: now reaches U3.25 (PB1)
- net PYRO1_FIRE: now reaches U3.5 (PH0)
- new net ADC1_IN6: U3.15 (PA1)
- no-connect marks 30 -> 23
