File: pcb/control-module.kicad_sch (KiCad schematic)
At the start: 21 parts, among them J1 Screw_Terminal_01x08, J2 Conn_01x06_Pin, J5 Screw_Terminal_01x02, SW1 SW_DIP_x03, U1 TC2185-3.3VxCTTR

Commit message: Revision 1
Parts:
- removed R4, R5, R6: 10k, Resistor_SMD:R_0603_1608Metric_Pad0.98x0.95mm_HandSolder, symbol Device:R_US
- added D4: B350A-13-F, Diode_SMD:D_SOD-123F, symbol Device:D
- added JP2: SolderJumper_2_Open, Jumper:SolderJumper-2_P1.3mm_Open_RoundedPad1.0x1.5mm, symbol Jumper:SolderJumper_2_Open
- added RN1, RN2: 10k, Resistor_SMD:R_Array_Convex_4x0612, symbol Device:R_Pack04
- J1: value Screw_Terminal_01x08 -> Screw_Terminal_01x06
- J2: value Conn_01x06_Pin -> Conn_01x07_Pin; footprint Connector_PinHeader_2.54mm:PinHeader_1x06_P2.54mm_Vertical -> Connector_PinHeader_2.54mm:PinHeader_1x07_P2.54mm_Vertical; symbol Connector:Conn_01x06_Pin -> Connector:Conn_01x07_Pin
- SW1: value SW_DIP_x03 -> SW_DIP_x04
Connections:
- net +3.3V: now also JP2.1 (A), RN2.1 (R1.1)
- net BOOT0: now also RN2.7 (R2.2)
- net GNDA: now also J2.7 (Pin_7), RN1.4 (R4.1); no longer J2.5 (Pin_5)
- net GNDD: now also RN2.2 (R2.1), RN2.3 (R3.1), RN2.4 (R4.1)
- net NRST: now also RN2.8 (R1.2)
- net Recovery Power: now also D4.1 (K)
- net SD_EJECT: now also RN2.6 (R3.2)
- net Valve Controller/Out: now also D4.2 (A)
- net at SW1.5: now also RN2.5 (R4.2)
- new net: RN1.2 (R2.1), RN1.3 (R3.1)
- new net: RN1.7 (R2.2), RN1.8 (R1.2)
- new net +BATT: J2.5 (Pin_5), RN1.1 (R1.1)
- new net Bat Sense: RN1.5 (R4.2), RN1.6 (R3.2)
- new net VDDA: JP2.2 (B)
- no-connect marks 2 -> 4
Other:
- sheet MCU ports: added ADC1_IN15, ADC1_IN16, ADC1_IN5, ADC1_IN6, PYRO1_FIRE, PYRO2_FIRE, VALVE_FIRE; removed SD_DAT1, SD_DAT2, SD_DAT3
- note added: "3.3V Indicator"
- note added: "Divide battery voltage by four to fit in ADC range. Will by multiplied by 4 in software."
- note added: "Only using 1-bit now"
- note added: "USB Voltage Regulator"
- moved on the sheet: C1, C2, C3, D2, JP1, R3, U1
